File: BMS/BMS.kicad_pcb (KiCad board)
At the start: 2 copper layers, 57.4 x 167.7 mm, 5 parts

Commit message: Update BMS.kicad_pcb
BMS packaging on the old board form factor.
Parts:
- added C1: 100nF, Capacitor_SMD:C_0805_2012Metric_Pad1.18x1.45mm_HandSolder, F.Cu at (50.5, 47.1)
- added C10: 10nF, Capacitor_SMD:C_0805_2012Metric_Pad1.18x1.45mm_HandSolder, F.Cu at (59.7, 132.5)
- added C11: 10nF, Capacitor_SMD:C_0805_2012Metric_Pad1.18x1.45mm_HandSolder, F.Cu at (59.9, 61.9)
- added C12: 15pF, Capacitor_SMD:C_0805_2012Metric_Pad1.18x1.45mm_HandSolder, F.Cu at (48.4, 119.2)
- added C13: 10nF, Capacitor_SMD:C_0805_2012Metric_Pad1.18x1.45mm_HandSolder, F.Cu at (50.9, 119.2)
- added C14: 10nF, Capacitor_SMD:C_0805_2012Metric_Pad1.18x1.45mm_HandSolder, F.Cu at (58.1, 38.6)
- added C2: 10nF, Capacitor_SMD:C_0805_2012Metric_Pad1.18x1.45mm_HandSolder, F.Cu at (58.9, 42.6)
- added C3: 1uF, Capacitor_SMD:C_0805_2012Metric_Pad1.18x1.45mm_HandSolder, F.Cu at (52.5, 47.1)
- added C5: 10nF, Capacitor_SMD:C_0805_2012Metric_Pad1.18x1.45mm_HandSolder, F.Cu at (42.1, 52.4)
- added C6: 1uF, Capacitor_SMD:C_0805_2012Metric_Pad1.18x1.45mm_HandSolder, F.Cu at (50.4, 84.7)
- added C7: 1uF, Capacitor_SMD:C_0805_2012Metric_Pad1.18x1.45mm_HandSolder, F.Cu at (50.4, 86.7)
- added C8: 10nF, Capacitor_SMD:C_0805_2012Metric_Pad1.18x1.45mm_HandSolder, F.Cu at (41.1, 123.2)
- added C9: 10nF, Capacitor_SMD:C_0805_2012Metric_Pad1.18x1.45mm_HandSolder, F.Cu at (48.3, 166.7)
- added D1: LH R974-LP-1, LED_SMD:LED_0805_2012Metric_Pad1.15x1.40mm_HandSolder, F.Cu at (49.7, 114.7)
- added D3: LH R974-LP-1, LED_SMD:LED_0805_2012Metric_Pad1.15x1.40mm_HandSolder, F.Cu at (36.6, 58.6)
- added D4: LH R974-LP-1, LED_SMD:LED_0805_2012Metric_Pad1.15x1.40mm_HandSolder, F.Cu at (36.0, 132.7)
- added D5: LH R974-LP-1, LED_SMD:LED_0805_2012Metric_Pad1.15x1.40mm_HandSolder, F.Cu at (55.1, 176.2)
- added D6: LH R974-LP-1, LED_SMD:LED_0805_2012Metric_Pad1.15x1.40mm_HandSolder, F.Cu at (62.1, 120.9)
- added D7: LH R974-LP-1, LED_SMD:LED_0805_2012Metric_Pad1.15x1.40mm_HandSolder, F.Cu at (63.4, 49.9)
- added D8: LH R974-LP-1, LED_SMD:LED_0805_2012Metric_Pad1.15x1.40mm_HandSolder, F.Cu at (50.4, 30.6)
- added D9: LH R974-LP-1, LED_SMD:LED_0805_2012Metric_Pad1.15x1.40mm_HandSolder, F.Cu at (50.4, 82.7)
- added F1: Polyfuse, Fuse:Fuse_1812_4532Metric_Pad1.30x3.40mm_HandSolder, F.Cu at (49.4, 35.1)
- added F2: Polyfuse, Fuse:Fuse_1812_4532Metric_Pad1.30x3.40mm_HandSolder, F.Cu at (67.9, 49.4)
- added F3: Polyfuse, Fuse:Fuse_1812_4532Metric_Pad1.30x3.40mm_HandSolder, F.Cu at (76.2, 122.7)
- added F4: Polyfuse, Fuse:Fuse_1812_4532Metric_Pad1.30x3.40mm_HandSolder, F.Cu at (56.9, 180.7)
- added F5: Polyfuse, Fuse:Fuse_1812_4532Metric_Pad1.30x3.40mm_HandSolder, F.Cu at (25.6, 127.4)
- added F6: Polyfuse, Fuse:Fuse_1812_4532Metric_Pad1.30x3.40mm_HandSolder, F.Cu at (30.4, 61.6)
- added F7: Polyfuse, Fuse:Fuse_1812_4532Metric_Pad1.30x3.40mm_HandSolder, F.Cu at (42.9, 47.4)
- added J1: Conn_01x02_Pin, Connector_Molex:Molex_Nano-Fit_105313-xx02_1x02_P2.50mm_Horizontal, F.Cu at (42.6, 42.6)
- added J2: IsoSPI, Connector_Molex:Molex_Nano-Fit_105313-xx02_1x02_P2.50mm_Horizontal, F.Cu at (49.0, 151.4)
- added J3: IsoSPI, Connector_Molex:Molex_Nano-Fit_105313-xx02_1x02_P2.50mm_Horizontal, F.Cu at (52.8, 146.9)
- added J4: ~, Connector_JST:JST_XH_S2B-XH-A_1x02_P2.50mm_Horizontal, F.Cu at (62.5, 88.2)
- added J5: ~, Connector_JST:JST_XH_S2B-XH-A_1x02_P2.50mm_Horizontal, F.Cu at (62.5, 96.6)
- added J6: ~, Connector_JST:JST_XH_S2B-XH-A_1x02_P2.50mm_Horizontal, F.Cu at (62.5, 162.4)
- added J7: ~, Connector_JST:JST_XH_S2B-XH-A_1x02_P2.50mm_Horizontal, F.Cu at (39.2, 159.9)
- added J8: ~, Connector_JST:JST_XH_S2B-XH-A_1x02_P2.50mm_Horizontal, F.Cu at (39.2, 94.0)
- added J9: ~, Connector_JST:JST_XH_S2B-XH-A_1x02_P2.50mm_Horizontal, F.Cu at (39.2, 85.7)
- added L1: HM2113ZNL, FS_3_Global_Footprint_Library:HM2113ZNLT, F.Cu at (50.9, 130.3)
- added Q1: NSV1C201MZ4, Package_TO_SOT_SMD:SOT-223, F.Cu at (50.0, 54.3)
- added Q3: BSS308PE, Package_TO_SOT_SMD:SOT-23, F.Cu at (38.4, 55.4)
- added Q4: BSS308PE, Package_TO_SOT_SMD:SOT-23, F.Cu at (38.0, 119.3)
- added Q5: BSS308PE, Package_TO_SOT_SMD:SOT-23, F.Cu at (51.6, 170.3)
- added Q6: BSS308PE, Package_TO_SOT_SMD:SOT-23, F.Cu at (63.7, 129.5)
- added Q7: BSS308PE, Package_TO_SOT_SMD:SOT-23, F.Cu at (63.5, 58.2)
- added Q8: BSS308PE, Package_TO_SOT_SMD:SOT-23, F.Cu at (58.4, 31.7)
- added R1: 100, Resistor_SMD:R_0805_2012Metric_Pad1.20x1.40mm_HandSolder, F.Cu at (47.1, 49.6)
- added R12: 1.5k, Resistor_SMD:R_0805_2012Metric_Pad1.20x1.40mm_HandSolder, F.Cu at (53.9, 63.4)
- added R13: 680, Resistor_SMD:R_0805_2012Metric_Pad1.20x1.40mm_HandSolder, F.Cu at (53.9, 61.4)
- added R15: 120, Resistor_SMD:R_0805_2012Metric_Pad1.20x1.40mm_HandSolder, F.Cu at (40.4, 58.6)
- added R16: 33, Resistor_SMD:R_2512_6332Metric_Pad1.40x3.35mm_HandSolder, F.Cu at (38.4, 61.6)
- added R17: 3.3k, Resistor_SMD:R_0805_2012Metric_Pad1.20x1.40mm_HandSolder, F.Cu at (41.1, 55.4)
- added R18: 100, Resistor_SMD:R_0805_2012Metric_Pad1.20x1.40mm_HandSolder, F.Cu at (38.4, 52.4)
- added R19: 120, Resistor_SMD:R_0805_2012Metric_Pad1.20x1.40mm_HandSolder, F.Cu at (39.7, 132.7)
- added R2: 100, Resistor_SMD:R_0805_2012Metric_Pad1.20x1.40mm_HandSolder, F.Cu at (47.1, 47.4)
- added R20: 33, Resistor_SMD:R_2512_6332Metric_Pad1.40x3.35mm_HandSolder, F.Cu at (38.0, 129.7)
- added R21: 3.3k, Resistor_SMD:R_0805_2012Metric_Pad1.20x1.40mm_HandSolder, F.Cu at (38.9, 123.2)
- added R22: 100, Resistor_SMD:R_0805_2012Metric_Pad1.20x1.40mm_HandSolder, F.Cu at (41.1, 119.2)
- added R23: 120, Resistor_SMD:R_0805_2012Metric_Pad1.20x1.40mm_HandSolder, F.Cu at (55.1, 172.4)
- added R24: 33, Resistor_SMD:R_2512_6332Metric_Pad1.40x3.35mm_HandSolder, F.Cu at (58.1, 174.4)
- added R25: 3.3k, Resistor_SMD:R_0805_2012Metric_Pad1.20x1.40mm_HandSolder, F.Cu at (51.5, 167.4)
- added R26: 100, Resistor_SMD:R_0805_2012Metric_Pad1.20x1.40mm_HandSolder, F.Cu at (48.3, 170.4)
- added R27: 120, Resistor_SMD:R_0805_2012Metric_Pad1.20x1.40mm_HandSolder, F.Cu at (62.1, 124.7)
- added R28: 33, Resistor_SMD:R_2512_6332Metric_Pad1.40x3.35mm_HandSolder, F.Cu at (65.2, 122.9)
- added R29: 3.3k, Resistor_SMD:R_0805_2012Metric_Pad1.20x1.40mm_HandSolder, F.Cu at (60.1, 130.4)
- added R3: 100, Capacitor_SMD:C_0805_2012Metric_Pad1.18x1.45mm_HandSolder, F.Cu at (56.9, 42.6)
- added R30: 100, Resistor_SMD:R_0805_2012Metric_Pad1.20x1.40mm_HandSolder, F.Cu at (63.6, 132.5)
- added R31: 120, Resistor_SMD:R_0805_2012Metric_Pad1.20x1.40mm_HandSolder, F.Cu at (63.4, 53.6)
- added R32: 402, Resistor_SMD:R_0805_2012Metric_Pad1.20x1.40mm_HandSolder, F.Cu at (53.4, 119.2)
- added R33: 2.2k, Resistor_SMD:R_0805_2012Metric_Pad1.20x1.40mm_HandSolder, F.Cu at (55.0, 99.0)
- added R34: 33, Resistor_SMD:R_2512_6332Metric_Pad1.40x3.35mm_HandSolder, F.Cu at (60.4, 51.9)
- added R35: 3.3k, Resistor_SMD:R_0805_2012Metric_Pad1.20x1.40mm_HandSolder, F.Cu at (59.6, 59.1)
- added R36: 100, Resistor_SMD:R_0805_2012Metric_Pad1.20x1.40mm_HandSolder, F.Cu at (63.6, 61.9)
- added R37: 10k, Resistor_SMD:R_0805_2012Metric_Pad1.20x1.40mm_HandSolder, F.Cu at (47.4, 100.9)
- added R38: 10k, Resistor_SMD:R_0805_2012Metric_Pad1.20x1.40mm_HandSolder, F.Cu at (48.6, 91.2)
- added R39: 10k, Resistor_SMD:R_0805_2012Metric_Pad1.20x1.40mm_HandSolder, F.Cu at (50.6, 91.2)
- added R4: 10k, Resistor_SMD:R_0805_2012Metric_Pad1.20x1.40mm_HandSolder, F.Cu at (56.1, 109.4)
- added R40: 22, Resistor_SMD:R_0805_2012Metric_Pad1.20x1.40mm_HandSolder, F.Cu at (52.6, 141.2)
- added R41: 22, Resistor_SMD:R_0805_2012Metric_Pad1.20x1.40mm_HandSolder, F.Cu at (48.1, 141.2)
- added R42: 120, Resistor_SMD:R_0805_2012Metric_Pad1.20x1.40mm_HandSolder, F.Cu at (54.1, 30.6)
- added R43: 33, Resistor_SMD:R_2512_6332Metric_Pad1.40x3.35mm_HandSolder, F.Cu at (52.1, 27.6)
- added R44: 3.3k, Resistor_SMD:R_0805_2012Metric_Pad1.20x1.40mm_HandSolder, F.Cu at (55.4, 34.9)
- added R45: 100, Resistor_SMD:R_0805_2012Metric_Pad1.20x1.40mm_HandSolder, F.Cu at (59.1, 35.6)
- added R5: 200, Resistor_SMD:R_0805_2012Metric_Pad1.20x1.40mm_HandSolder, F.Cu at (46.4, 116.9)
- added R51: 160, Resistor_SMD:R_0805_2012Metric_Pad1.20x1.40mm_HandSolder, F.Cu at (53.4, 83.7)
- added R6: 160, Resistor_SMD:R_0805_2012Metric_Pad1.20x1.40mm_HandSolder, F.Cu at (49.6, 112.7)
- added R7: 10k, Resistor_SMD:R_0805_2012Metric_Pad1.20x1.40mm_HandSolder, F.Cu at (56.1, 107.4)
- added R8: 10k, Resistor_SMD:R_0805_2012Metric_Pad1.20x1.40mm_HandSolder, F.Cu at (56.1, 105.4)
- added SW2: A6H-4101, FS_3_Global_Footprint_Library:SW_A6H-4101_OMR, F.Cu at (50.1, 107.8)
- added U2: ADG708, Package_SO:TSSOP-16_4.4x5mm_P0.65mm, F.Cu at (51.2, 97.0)
- added U3: LTC6811IG-2-TRPBF, FS_3_Global_Footprint_Library:LTC6811-2, F.Cu at (50.8, 72.2)
Routing:
- net /C3: track 0.00 -> 122.3 mm
- net VREG: track 0.00 -> 113.8 mm, vias 0 -> 2
- net /C7: track 0.00 -> 104.6 mm
- net /S7: track 0.00 -> 101.9 mm
- net /C2: track 0.00 -> 100.3 mm
- net /BB1/B#+1: track 0.00 -> 77.4 mm
- net /C8: track 0.00 -> 74.7 mm
- net /BB4/B#+1: track 0.00 -> 72.2 mm
- net /S3: track 0.00 -> 71.3 mm
- net Net-(J7-Pin_2): track 0.00 -> 69.3 mm, vias 0 -> 1
- net /BB3/B#+1: track 0.00 -> 65.1 mm
- net Net-(J6-Pin_2): track 0.00 -> 65.1 mm, vias 0 -> 1
- net IsoSPI_P: track 0.00 -> 59.9 mm
- net IsoSPI_N: track 0.00 -> 59.3 mm
- net /BB2/B#+1: track 0.00 -> 58.7 mm
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- added copper zone on B.Cu, net V-

Commit message: Update BMS.kicad_pcb
Other:
- board size 57.4 x 167.7 mm -> 57.4 x 171.2 mm

Commit message: Update BMS.kicad_pcb
updated J1-3 to fit the required 20mm clearances
Parts:
- moved R2 13.1 mm to (37.6, 56.3)
- moved R1 12.9 mm to (37.6, 58.3)
- moved J3 12.3 mm to (45.2, 156.5)
- moved J1 11.9 mm to (41.8, 54.5)
- moved C5 7.90 mm to (42.1, 60.3)
- moved Q3 7.90 mm to (38.4, 63.3)
- moved R17 7.90 mm to (41.1, 63.3)
- moved R18 7.90 mm to (38.4, 60.3)
- moved J2 7.90 mm to (56.5, 153.9)
- moved F7 7.82 mm to (36.6, 52.0)
- moved F3 7.27 mm to (69.7, 119.3), turned to -90 degrees
- moved D3 7.17 mm to (29.7, 60.5)
- moved R15 6.95 mm to (33.7, 60.5)
- moved R16 6.95 mm to (31.7, 63.5)
- moved F6 6.44 mm to (24.9, 58.3), turned to 90 degrees
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Routing:
- net /extIsoSPI_N: track 14.8 -> 35.2 mm
- net /BB3/B#+1: track 65.1 -> 52.8 mm
- net /extIsoSPI_P: track 16.9 -> 25.5 mm
- net /S9: track 28.5 -> 20.6 mm
- net /C9-12: track 30.7 -> 22.8 mm
- net /C8: track 74.7 -> 66.8 mm
- net VREG: track 113.8 -> 121.3 mm
- net Net-(C1-Pad1): track 15.1 -> 22.3 mm
- net Net-(J1-Pin_2): track 8.03 -> 15.2 mm
- net Net-(F3-Pad2): track 10.5 -> 4.66 mm
- net /BB2/B#+1: track 58.7 -> 53.3 mm
- net /BB5/B#+1: track 14.7 -> 9.69 mm
- net /DRV: track 20.2 -> 25.0 mm
- net Net-(J1-Pin_1): track 2.65 -> 7.16 mm
- net /BB1/B#+1: track 77.4 -> 73.2 mm
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